File: Temperature.kicad_sch (KiCad schematic)
At the start: 6 parts

Commit message: 0.2: флаги питания расставлены в GUI, ERC 19 -> 9
Десять PWR_FLAG (#FLG1..#FLG10) поставлены в редакторе на цепи +3.3V,
+3.3VA, VDC, +12V, три локальные цепи за FB7..FB9 (один флаг в
Temperature.kicad_sch покрыл все три экземпляра) и три за FB10..FB12 в
Current_Sensor_1/2/3. Добавлены сопутствующие символы шин
(#PWR50-51, #PWR93).

Проверено:
- ERC 19 -> 9 ошибок, power_pin_not_driven 11 -> 1 (осталась GND);
- hier_label_mismatch нет — иерархия в порядке, в отличие от того, что
  получалось при моих попытках правки файлов текстом;
- netlist совпадает с исходным байт в байт, кроме двух строк pintype у
  J6.14/16 от моего no_connect: связность не изменилась ни в одной цепи;
- DRC 0 нарушений, 0 неподключённых, 0 расхождений со схемой.

Уточнение, снимающее мою прежнюю ошибку в диагностике: символы питания
(#PWR*, #FLG*) в netlist не попадают вообще — в netlist ноль вхождений
#PWR. Так что отсутствие флагов в netlist не было признаком поломки;
признаком были hier_label_mismatch и потеря ~30 КБ содержимого.

В CHANGELOG сведён остаток 0.2: флаг на GND, 8 ошибок по символу
TLV3502AIDR (уйдут с U6 по §3.1), 17 lib_symbol_mismatch, 12
endpoint_off_grid (в §1.3) и метка DAC_1_MCU, по которой нужно решение.

Co-Authored-By: Claude Opus 5 <noreply@anthropic.com>
Changed lines of the file:
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@@
+	)
+	(symbol
+		(lib_id "power:PWR_FLAG")
+		(at 138.43 91.44 90)
+		(unit 1)
+		(body_style 1)
+		(exclude_from_sim no)
+		(in_bom yes)
+		(on_board yes)
+		(in_pos_files yes)
+		(dnp no)
+		(fields_autoplaced yes)
+		(property "Reference" "#FLG03"
+			(at 136.525 91.44 0)
+			(hide yes)
+			(show_name no)
+			(do_not_autoplace no)
+			(effects
+				(font
+					(size 1.27 1.27)
+				)
+			)
+		)
+		(property "Value" "PWR_FLAG"
+			(at 134.62 91.4399 90)
+			(show_name no)
+			(do_not_autoplace no)
+			(effects
+				(font
+					(size 1.27 1.27)
+				)
+				(justify left)
+			)
+		)
+		(property "Footprint" ""
+			(at 138.43 91.44 0)
+			(hide yes)
+			(show_name no)
+			(do_not_autoplace no)
+			(effects
+				(font
+					(size 1.27 1.27)
+				)
+			)
+		)
+		(property "Datasheet" ""
+			(at 138.43 91.44 0)
+			(hide yes)
+			(show_name no)
+			(do_not_autoplace no)
+			(effects
+				(font
+					(size 1.27 1.27)
+				)
+			)
+		)
+		(property "Description" "Special symbol for telling ERC where power comes from"
+			(at 138.43 91.44 0)
+			(hide yes)
+			(show_name no)
+			(do_not_autoplace no)
+			(effects
+				(font
+					(size 1.27 1.27)
+				)
+			)
+		)
+		(pin "1"
+		)
+		(instances
+			(project "Power"
+				(path "/7ff38f8b-11c9-43a1-8b76-b5e8c8de18e0/920de354-6a24-4ec8-b59a-17ed91dfdddb"
+					(reference "#FLG03")
+					(unit 1)
+				)
+				(path "/7ff38f8b-11c9-43a1-8b76-b5e8c8de18e0/d6af5e0c-29a9-4f29-a8a0-ace2d5817bf6"
+					(reference "#FLG05")
+					(unit 1)
+				)
+				(path "/7ff38f8b-11c9-43a1-8b76-b5e8c8de18e0/e9b86447-9b47-4c39-b0c9-de73fedf4620"
+					(reference "#FLG04")
+					(unit 1)
+				)
+			)
+		)
 	)
 	(symbol
