File: Power.kicad_sch (KiCad schematic)
At the start: 106 parts, among them Y1 16M

Commit message: §1.5: контур расширяется до 60 мм, раскладка 2x3 с осью тока вдоль x
Решение от 2026-10-09: плату расширяем. Раздел переписан от требований.

Поправка к прежнему расчёту: полосу по y ограничивают не электролиты
(их пэды кончаются на y = 67,6), а СУЖЕНИЕ КОНТУРА — прямые участки
боковых кромок идут только от y = 71,5 до y = 92,8. Полоса на полную
ширину 53,0 x 21,0 = 1113 мм2 против 1086 мм2 шести корпусов, то есть
заполнение 97,6 % и нуль свободного места.

Ограничение по y окончательное: вертикальная ось тока просит 35,5 мм,
а нарастить полосу можно максимум до 22,2 (плата 108,76 при радиаторе
110). Одиночный ряд из шести с вертикальной осью даёт поле приборов
63,7 мм против 63 мм радиатора. Значит 2 ряда по 3 с осью тока вдоль x
— единственный вариант, фиксируется окончательно.

Электрическая раскладка: ряд HS сверху, ряд LS снизу зеркально, узел
фазы собирается на правом торце пары (исток HS прямо над стоком LS),
VDC и GND приходят на левый торец снизу из In1/In2 через виа. Петля
одной фазы ~17,7 x 11 мм, обратный ток по In4 в 0,1 мм.

Бюджет по y требует выпрямить скругления вверху до y = 68,5: тогда
24,0 мм раскладываются как 1,8 (обвязка HS) + 10,2 + 0,5 + 10,2 + 1,3
(обвязка LS). Полоски 1,3..1,8 мм вмещают SOT-23 и 0603, то есть кламп
Миллера встаёт вплотную к выводам G/S без виа в контуре, как требует
§1.4. Без выпрямления этого места нет.

Бюджет по x: рекомендована ширина платы 60 мм (поле приборов 58,2 при
радиаторе 63, по 2,4 мм с каждой стороны).

Новое следствие: шаг пар 19,05 мм против шага втулок J1..J3 12,00 мм —
расхождение 7 мм, фазный ток 500 A придётся сводить с боковым
смещением по внутренним слоям. Вынесен вопрос, можно ли сдвинуть
втулки под новый шаг.

Co-Authored-By: Claude Opus 5 <noreply@anthropic.com>
Changed lines of the file:
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@@
 	)
 	(junction
+		(at 359.41 203.2)
+		(diameter 0)
+		(color 0 0 0 0)
+	)
+	(junction
 		(at 505.46 198.12)
 		(diameter 0)
@@
 	(wire
 		(pts
+			(xy 359.41 204.47) (xy 359.41 203.2)
+		)
+		(stroke
+			(width 0)
+			(type default)
+		)
+	)
+	(wire
+		(pts
 			(xy 91.44 140.97) (xy 100.33 140.97)
 		)
@@
 	(wire
 		(pts
+			(xy 359.41 203.2) (xy 359.41 200.66)
+		)
+		(stroke
+			(width 0)
+			(type default)
+		)
+	)
+	(wire
+		(pts
 			(xy 341.63 195.58) (xy 359.41 195.58)
 		)
@@
 	)
 	(symbol
+		(lib_id "power:PWR_FLAG")
+		(at 359.41 203.2 90)
+		(unit 1)
+		(body_style 1)
+		(exclude_from_sim no)
+		(in_bom yes)
+		(on_board yes)
+		(in_pos_files yes)
+		(dnp no)
+		(fields_autoplaced yes)
+		(property "Reference" "#FLG011"
+			(at 357.505 203.2 0)
+			(hide yes)
+			(show_name no)
+			(do_not_autoplace no)
+			(effects
+				(font
+					(size 1.27 1.27)
+				)
+			)
+		)
+		(property "Value" "PWR_FLAG"
+			(at 355.6 203.1999 90)
+			(show_name no)
+			(do_not_autoplace no)
+			(effects
+				(font
+					(size 1.27 1.27)
+				)
+				(justify left)
+			)
+		)
+		(property "Footprint" ""
+			(at 359.41 203.2 0)
+			(hide yes)
+			(show_name no)
+			(do_not_autoplace no)
+			(effects
+				(font
+					(size 1.27 1.27)
+				)
+			)
+		)
+		(property "Datasheet" ""
+			(at 359.41 203.2 0)
+			(hide yes)
+			(show_name no)
+			(do_not_autoplace no)
+			(effects
+				(font
+					(size 1.27 1.27)
+				)
+			)
+		)
+		(property "Description" "Special symbol for telling ERC where power comes from"
+			(at 359.41 203.2 0)
+			(hide yes)
+			(show_name no)
+			(do_not_autoplace no)
+			(effects
+				(font
+					(size 1.27 1.27)
+				)
+			)
+		)
+		(pin "1"
+		)
+		(instances
+			(project "Power"
+				(path "/7ff38f8b-11c9-43a1-8b76-b5e8c8de18e0"
+					(reference "#FLG011")
+					(unit 1)
+				)
+			)
+		)
+	)
+	(symbol
 		(lib_id "power:GND")
 		(at 414.02 212.09 0)
@@
 	(symbol
 		(lib_id "power:GND")
-		(at 359.41 200.66 0)
+		(at 359.41 204.47 0)
 		(unit 1)
 		(body_style 1)
@@
 		(dnp no)
 		(property "Reference" "#PWR0148"
-			(at 359.41 207.01 0)
+			(at 359.41 210.82 0)
 			(hide yes)
 			(show_name no)
@@
 		)
 		(property "Value" "GND"
-			(at 359.41 204.216 0)
+			(at 359.41 208.026 0)
 			(show_name no)
 			(do_not_autoplace no)
@@
 		)
 		(property "Footprint" ""
-			(at 359.41 200.66 0)
+			(at 359.41 204.47 0)
 			(hide yes)
 			(show_name no)
@@
 		)
 		(property "Datasheet" ""
-			(at 359.41 200.66 0)
+			(at 359.41 204.47 0)
 			(hide yes)
 			(show_name no)
@@
 		)
 		(property "Description" ""
-			(at 359.41 200.66 0)
+			(at 359.41 204.47 0)
 			(hide yes)
 			(show_name no)
