File: Power.kicad_sch (KiCad schematic)
At the start: 111 parts, among them Y1 16M

Commit message: Правки владельца: R8 (0603) последовательно в DAC_1_MCU на B.Cu у TP1, трасса DAC перезаведена по B.Cu; порядок листов и Power.kicad_pro пересохранены KiCad
Co-Authored-By: Claude Opus 5.5 <noreply@anthropic.com>
Parts:
- added R8: R, Resistor_SMD:R_0603_1608Metric_Pad0.98x0.95mm_HandSolder, symbol Device:R
Connections:
- net DAC_1_MCU: now also R8.1; no longer TP1.1
- new net: R8.2, TP1.1

Commit message: rev0.1-adapto: габарит и верхняя зона ADAPTO на 3 мм выше (V1, 53 × 101 мм, lay_AD1.py) и Y-цепь корпуса по docs/Y_TASK.md у H2 (fp_y.py, sch_rev01_j.py, lay_Y1.py; конвейер adapto.sh)
- вместо H5 и пары C135 / C136 одна цепь CHASSIS-CY1-CY2-FY1-GND и RY1-RY2 на B.Cu у правого U-паза H2 (H_CHS, подкова на F/B/In1-In4, 9 виа)
- netclass Y_CHASSIS и правила 0.5 / 0.8 / 2 мм; ISO / CHS на шелкографии; MPN, Alt_MPN, Note, Variant
- отчёт docs/REV1_Y_REPORT.md, вопросы docs/REV1_QUESTIONS.md, проверки y_checks.py
- DRC 0 / 0 / 0, ERC 9 (база), hv.py 23

Co-Authored-By: Claude Opus 5.5 <noreply@anthropic.com>
Parts:
- removed C135, C136: 4.7n Y2, Capacitor_SMD:C_1812_4532Metric, symbol Device:C_Small
- removed H2: MountingHole, MountingHole:MountingHole_3.2mm_M3, symbol Mechanical:MountingHole
- removed H5: MountingHole_Pad, MountingHole:MountingHole_3.2mm_M3_Pad_Via, symbol Mechanical:MountingHole_Pad
- added CY1, CY2: 470n 250V X7R, Capacitor_SMD:C_1812_4532Metric, symbol Device:C_Small
- added FY1: 2A 125VDC, Power_My:Fuse_2410_1206, symbol Device:Fuse_Small
- added H2: H_CHS, Power_My:MountingHole_3.2mm_M3_Slot_CHS, symbol Mechanical:MountingHole_Pad
- added RY1, RY2: 100k, Resistor_SMD:R_0805_2012Metric, symbol Device:R_Small
- added TP2: TP_CHS, TestPoint:TestPoint_Pad_D1.5mm, symbol Connector:TestPoint
- added TP3: TP_GND, TestPoint:TestPoint_Pad_D1.5mm, symbol Connector:TestPoint
Connections:
- net CHASSIS: now also CY1.1, H2.1, RY1.1, TP2.1
- net GND: now also FY1.1, RY2.2, TP3.1
- new net CY_MID: CY1.2, CY2.1
- new net RY_MID: RY1.2, RY2.1
- new net Y_F: CY2.2, FY1.2
Other:
- note added: "Y-цепь корпуса"
- note added: "Минус ЗПТ - радиатор (корпус), docs/Y_TASK.md: возврат синфазного тока коротким путём, потенциал корпуса без связи по постоянному току, путь ESD. Одна цепь от минуса: вторую цепь от +DC не ставить. H2 - винт в радиатор, кольцо CHASSIS (шайба зубчатая или пружинная); H1, H3, H4 - без меди под шайбой. CY1, CY2: 250 V, soft termination - не заменять на 100 V. RY1, RY2 - мимо FY1: при сгоревшем FY1 к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"
