File: Current_Sensor_3.kicad_sch (KiCad schematic)
At the start: 6 parts

Commit message: 0.2: флаги питания расставлены в GUI, ERC 19 -> 9
Десять PWR_FLAG (#FLG1..#FLG10) поставлены в редакторе на цепи +3.3V,
+3.3VA, VDC, +12V, три локальные цепи за FB7..FB9 (один флаг в
Temperature.kicad_sch покрыл все три экземпляра) и три за FB10..FB12 в
Current_Sensor_1/2/3. Добавлены сопутствующие символы шин
(#PWR50-51, #PWR93).

Проверено:
- ERC 19 -> 9 ошибок, power_pin_not_driven 11 -> 1 (осталась GND);
- hier_label_mismatch нет — иерархия в порядке, в отличие от того, что
  получалось при моих попытках правки файлов текстом;
- netlist совпадает с исходным байт в байт, кроме двух строк pintype у
  J6.14/16 от моего no_connect: связность не изменилась ни в одной цепи;
- DRC 0 нарушений, 0 неподключённых, 0 расхождений со схемой.

Уточнение, снимающее мою прежнюю ошибку в диагностике: символы питания
(#PWR*, #FLG*) в netlist не попадают вообще — в netlist ноль вхождений
#PWR. Так что отсутствие флагов в netlist не было признаком поломки;
признаком были hier_label_mismatch и потеря ~30 КБ содержимого.

В CHANGELOG сведён остаток 0.2: флаг на GND, 8 ошибок по символу
TLV3502AIDR (уйдут с U6 по §3.1), 17 lib_symbol_mismatch, 12
endpoint_off_grid (в §1.3) и метка DAC_1_MCU, по которой нужно решение.

Co-Authored-By: Claude Opus 5 <noreply@anthropic.com>
Changed lines of the file:
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@@
+	)
+	(symbol
+		(lib_id "power:PWR_FLAG")
+		(at 127 111.76 90)
+		(unit 1)
+		(body_style 1)
+		(exclude_from_sim no)
+		(in_bom yes)
+		(on_board yes)
+		(in_pos_files yes)
+		(dnp no)
+		(fields_autoplaced yes)
+		(property "Reference" "#FLG08"
+			(at 125.095 111.76 0)
+			(hide yes)
+			(show_name no)
+			(do_not_autoplace no)
+			(effects
+				(font
+					(size 1.27 1.27)
+				)
+			)
+		)
+		(property "Value" "PWR_FLAG"
+			(at 123.19 111.7599 90)
+			(show_name no)
+			(do_not_autoplace no)
+			(effects
+				(font
+					(size 1.27 1.27)
+				)
+				(justify left)
+			)
+		)
+		(property "Footprint" ""
+			(at 127 111.76 0)
+			(hide yes)
+			(show_name no)
+			(do_not_autoplace no)
+			(effects
+				(font
+					(size 1.27 1.27)
+				)
+			)
+		)
+		(property "Datasheet" ""
+			(at 127 111.76 0)
+			(hide yes)
+			(show_name no)
+			(do_not_autoplace no)
+			(effects
+				(font
+					(size 1.27 1.27)
+				)
+			)
+		)
+		(property "Description" "Special symbol for telling ERC where power comes from"
+			(at 127 111.76 0)
+			(hide yes)
+			(show_name no)
+			(do_not_autoplace no)
+			(effects
+				(font
+					(size 1.27 1.27)
+				)
+			)
+		)
+		(pin "1"
+		)
+		(instances
+			(project "Power"
+				(path "/7ff38f8b-11c9-43a1-8b76-b5e8c8de18e0/135c859b-ab7a-4fd9-b627-73749955badd"
+					(reference "#FLG08")
+					(unit 1)
+				)
+			)
+		)
 	)
 	(symbol

Commit message: Замечания владельца 19.10: все дорожки под 0/45/90° (octo.py, 76 отрезков); VDC на J6 от верхней полосы по In2, через проход C по In1 — In2 узла C в проходе одним куском; линии термистора C по In1 без виа в горле прохода; U4/U9/U12 — INA240A1 (пин в пин); DRC 0/0/0
Co-Authored-By: Claude Opus 5.5 <noreply@anthropic.com>
Parts:
- U12: symbol Amplifier_Current:AD8418 -> Logic_My:INA240A1D; Product Name AD8418 -> INA240A1DR
Changed lines of the file:
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@@
 	)
 	(symbol
-		(lib_id "Amplifier_Current:AD8418")
+		(lib_id "Logic_My:INA240A1D")
 		(at 143.51 109.22 0)
 		(unit 1)
@@
 			)
 		)
-		(property "Datasheet" "https://www.analog.com/media/en/technical-documentation/data-sheets/AD8418.pdf"
+		(property "Datasheet" "https://www.ti.com/lit/ds/symlink/ina240.pdf"
 			(at 160.02 127 0)
 			(hide yes)
@@
 			)
 		)
-		(property "Description" "70V Bidirectional, Zero Drift, Current Sense Amplifier, 20V/V gain, bandwidth 250kHz, VS=2.7V~5.5V, SOIC-8/MSOP-8"
+		(property "Description" "-4...80V Bidirectional, Zero Drift, Current Sense Amplifier With Enhanced PWM Rejection, 20V/V gain, bandwidth 400kHz, VS=2.7V~5.5V, SOIC-8 (pin compatible with AD8418)"
 			(at 143.51 109.22 0)
 			(hide yes)
@@
 			)
 		)
-		(property "Product Name" "AD8418"
+		(property "Product Name" "INA240A1DR"
 			(at 143.51 109.22 0)
 			(hide yes)

Commit message: Анализ растекания тока в силовой меди (cflow.py): узел → шунт, VDC, GND по фазам, ценность слоёв, предложенные виа сшивки (не применены); U4/U9/U12 — замена на INA241A2 при 72 В в поле Replacement; виа сшивки с (free yes); решения владельца по S3, E6, R снабберов
Co-Authored-By: Claude Opus 5.5 <noreply@anthropic.com>
Parts:
- U12: Replacement (none) -> INA241A2DR при VDC 72 В
Changed lines of the file:
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@@
 			)
 		)
-		(property "Replacement" ""
+		(property "Replacement" "INA241A2DR при VDC 72 В"
 			(at 143.51 109.22 0)
 			(hide yes)

Commit message: Ревью rev0.1-plus4, раунд 3 (11 силовик, 13 ЭМС): C134 100n 100V у J6 на B.Cu; C37/C39/C64 15n; R50 DNP; вывод 4 U4/U9/U12 на GND (под INA241A2); cflow исправлен — стакан связан с медью у стенки, сетка 0.05 мм, меры у шунта вместо пика (медь узла была занижена в 1.3–2.4 раза, решения в силе, фазы по меди равны 0.52–0.58 мОм); ответы 12/14; DRC 0/0/0
Co-Authored-By: Claude Opus 5.5 <noreply@anthropic.com>
Parts:
- C64: value 100n -> 15n
Connections:
- net GND: now also U12.4 (NC)
Changed lines of the file:
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@@
+	)
+	(symbol
+		(lib_id "power:GND")
+		(at 146.05 116.84 0)
+		(unit 1)
+		(body_style 1)
+		(exclude_from_sim no)
+		(in_bom yes)
+		(on_board yes)
+		(in_pos_files yes)
+		(dnp no)
+		(property "Reference" "#PWR220"
+			(at 146.05 123.19 0)
+			(hide yes)
+			(show_name no)
+			(do_not_autoplace no)
+			(effects
+				(font
+					(size 1.27 1.27)
+				)
+			)
+		)
+		(property "Value" "GND"
+			(at 146.05 120.65 0)
+			(show_name no)
+			(do_not_autoplace no)
+			(effects
+				(font
+					(size 1.27 1.27)
+				)
+			)
+		)
+		(property "Footprint" ""
+			(at 146.05 116.84 0)
+			(hide yes)
+			(show_name no)
+			(do_not_autoplace no)
+			(effects
+				(font
+					(size 1.27 1.27)
+				)
+			)
+		)
+		(property "Datasheet" ""
+			(at 146.05 116.84 0)
+			(hide yes)
+			(show_name no)
+			(do_not_autoplace no)
+			(effects
+				(font
+					(size 1.27 1.27)
+				)
+			)
+		)
+		(property "Description" ""
+			(at 146.05 116.84 0)
+			(hide yes)
+			(show_name no)
+			(do_not_autoplace no)
+			(effects
+				(font
+					(size 1.27 1.27)
+				)
+			)
+		)
+		(pin "1"
+		)
+		(instances
+			(project "Power"
+				(path "/7ff38f8b-11c9-43a1-8b76-b5e8c8de18e0/135c859b-ab7a-4fd9-b627-73749955badd"
+					(reference "#PWR220")
+					(unit 1)
+				)
+			)
+		)
 	)
 	(symbol
@@
 			)
 		)
-		(property "Value" "100n"
+		(property "Value" "15n"
 			(at 162.814 114.808 0)
 			(show_name no)
